Commit message: Temp 240315

File: grobot_description/urdf/grobot.urdf (robot description, URDF)
Before this commit: robot aedbot, 9 links, 8 joints
Links:
- link base_link: geometry collision mesh filename=package://grobot_description/meshes/bases/grobot_body.stl scale=0.001 0.001 0.001; visual mesh filename=package://aedbot_description/meshes/bases/grobot_body.stl scale=0.001 0.001 0.001
- link wheel_left_link: geometry collision mesh filename=package://grobot_description/meshes/wheels/grobot_wheel.stl scale=0.001 0.001 0.001; visual mesh filename=package://grobot_description/meshes/wheels/grobot_wheel.stl scale=0.001 0.001 0.001
- link wheel_right_link: geometry collision mesh filename=package://aedbot_description/meshes/wheels/aedbot_wheel.stl scale=0.001 0.001 0.001; visual mesh filename=package://grobot_description/meshes/wheels/aedbot_wheel.stl scale=0.001 0.001 0.001
