Commit message: Add grobot.xacro

File: grobot_description/urdf/grobot/grobot.xacro (robot description, xacro)
@@ -102,11 +102,11 @@
     <origin xyz="0.0 0.0 0.0" rpy="0 0 0"/>
     <geometry>
-      <cylinder length="0.0315" radius="0.055"/>
-    </geometry>
-  </collision>
-  <visual>
-    <origin xyz="0.0 0.0 0.0" rpy="0 0 0"/>
-    <geometry>
-      <cylinder length="0.0315" radius="0.055"/>
+      <cylinder length="0.0315" radius="0.035"/>
+    </geometry>
+  </collision>
+  <visual>
+    <origin xyz="0.0 0.0 0.0" rpy="0 0 0"/>
+    <geometry>
+      <cylinder length="0.0315" radius="0.035"/>
     </geometry>
   </visual>
@@ -128,11 +128,11 @@
     <origin xyz="0.0 0.0 0.0" rpy="0 0 0"/>
     <geometry>
-      <cylinder length="0.0315" radius="0.055"/>
-    </geometry>
-  </collision>
-  <visual>
-    <origin xyz="0.0 0.0 0.0" rpy="0 0 0"/>
-    <geometry>
-      <cylinder length="0.0315" radius="0.055"/>
+      <cylinder length="0.0315" radius="0.035"/>
+    </geometry>
+  </collision>
+  <visual>
+    <origin xyz="0.0 0.0 0.0" rpy="0 0 0"/>
+    <geometry>
+      <cylinder length="0.0315" radius="0.035"/>
     </geometry>
   </visual>
@@ -159,5 +159,5 @@
     <origin xyz="0.0 0.0 0.0" rpy="0 0 0"/>
     <geometry>
-      <cylinder length="0.0315" radius="0.055"/>
+      <cylinder length="0.0315" radius="0.035"/>
     </geometry>
   </visual>

Commit message: Add Camera Frame

File: grobot_description/urdf/grobot/grobot.xacro (robot description, xacro)
@@ -9,4 +9,11 @@
   <parent link="base_footprint"/>
   <child link="base_link"/>
+  <origin xyz="0 0.0 0.0" rpy="0 0 0.0"/>
+</joint>
+<!-- CAMERA LINK -->
+<link name="camera_link"/>
+<joint name="camera_joint" type="fixed">
+  <parent link="imu_link"/>
+  <child link="camera_link"/>
   <origin xyz="0 0.0 0.0" rpy="0 0 0.0"/>
 </joint>
