Commit message: Fix : URDF Wheel Axis

File: grobot_description/urdf/R1V2/R1V2.xacro (robot description, xacro)
@@ -68,5 +68,5 @@
   <parent link="base_link"/>
   <child link="right_wheel_1"/>
-  <axis xyz="0.0 -1.0 0.0"/>
+  <axis xyz="0.0 1.0 0.0"/>
 </joint>
 <joint name="left_wheel_joint" type="continuous">

Commit message: Add : Gazebo Cartographer

File: grobot_description/urdf/R1V2/R1V2.xacro (robot description, xacro)
@@ -4,4 +4,11 @@
 <xacro:include filename="$(find grobot_description)/urdf/R1V2.trans" />
 <xacro:include filename="$(find grobot_description)/urdf/R1V2.gazebo" />
+<xacro:property name="body_color" value="Gazebo/Grey" />
+<link name="base_footprint"/>
+<joint name="base_joint" type="fixed">
+  <parent link="base_footprint"/>
+  <child link="base_link"/>
+  <origin xyz="0 0.0 0.0" rpy="0 0 0.0"/>
+</joint>
 <link name="base_link">
   <inertial>
@@ -64,4 +71,23 @@
   </collision>
 </link>
+<link name="base_scan">
+  <inertial>
+    <origin xyz="0.0 0.0 0.0" rpy="0 0 0"/>
+    <mass value="0.114"/>
+    <inertia ixx="0.001" iyy="0.000000" izz="0.000000" ixy="0.001" iyz="0.000000" ixz="0.001"/>
+  </inertial>
+  <!-- <visual name="lidar_sensor_visual">
+    <origin xyz="0.0 0.0 0.0" rpy="0 0 0"/>
+    <geometry>
+      <mesh filename="file://$(find grobot_description)/meshes/lidar_1.stl" scale="0.001 0.001 0.001"/>
+    </geometry>
+  </visual>
+  <collision name="lidar_sensor_collision">
+    <origin xyz="0.0 0.0 0.0" rpy="0 0 0"/>
+    <geometry>
+      <mesh filename="file://$(find grobot_description)/meshes/lidar_1.stl" scale="0.001 0.001 0.001"/>
+    </geometry>
+  </collision> -->
+</link>
 <joint name="right_wheel_joint" type="continuous">
   <origin xyz="0.19013 -0.260644 0.100803" rpy="0 0 0"/>
@@ -76,4 +102,116 @@
   <axis xyz="0.0 1.0 -0.0"/>
 </joint>
+<joint name="lidar_joint" type="fixed">
+  <origin xyz="0.0 0.0 0.4" rpy="0 0 3.14159"/>
+  <parent link="base_link"/>
+  <child link="base_scan"/>
+  <axis xyz="0.0 0.0 1.0"/>
+</joint>
+<joint name="imu_joint" type="fixed">
+  <origin xyz="0.0 0.0 0.2" rpy="0 0 0"/>
+  <parent link="base_link"/>
+  <child link="imu_link"/>
+  <axis xyz="0.0 0.0 1.0"/>
+</joint>
+<gazebo reference="base_scan">
+        <sensor name="laser" type="ray">
+            <pose> 0 0 0 0 0 0 </pose>
+            <visualize>true</visualize>
+            <update_rate>10</update_rate>
+            <ray>
+                <scan>
+                    <horizontal>
+                        <samples>360</samples>
+                        <min_angle>-3.14</min_angle>
+                        <max_angle>3.14</max_angle>
+                    </horizontal>
+                </scan>
+                <range>
+                    <min>0.1</min>
+                    <max>16</max>
+                </range>
+                <noise>
+                  <type>gaussian</type>
+                  <mean>0.0</mean>
+                  <stddev>0.01</stddev>
+                </noise>
+            </ray>
+            <plugin name="scan" filename="libgazebo_ros_ray_sensor.so">
+                <ros>
+                    <argument>~/out:=scan</argument>
+                </ros>
+                <output_type>sensor_msgs/LaserScan</output_type>
+                <frame_name>base_scan</frame_name>
+            </plugin>
+        </sensor>
+</gazebo>
+<link name="imu_link"/>
+ <gazebo reference="imu_link">
+  <sensor name="imu_sensor" type="imu">
+   <plugin filename="libgazebo_ros_imu_sensor.so" name="imu_plugin">
+      <ros>
+        <remapping>~/out:=imu</remapping>
+      </ros>
+      <initial_orientation_as_reference>false</initial_orientation_as_reference>
+    </plugin>
+    <always_on>true</always_on>
+    <update_rate>100</update_rate>
+    <visualize>true</visualize>
+    <imu>
+      <angular_velocity>
+        <x>
+          <noise type="gaussian">
+            <mean>0.0</mean>
+            <stddev>2e-4</stddev>
+            <bias_mean>0.0000075</bias_mean>
+            <bias_stddev>0.0000008</bias_stddev>
+          </noise>
+        </x>
+        <y>
+          <noise type="gaussian">
+            <mean>0.0</mean>
+            <stddev>2e-4</stddev>
+            <bias_mean>0.0000075</bias_mean>
+            <bias_stddev>0.0000008</bias_stddev>
+          </noise>
+        </y>
+        <z>
+          <noise type="gaussian">
+            <mean>0.0</mean>
+            <stddev>2e-4</stddev>
+            <bias_mean>0.0000075</bias_mean>
+            <bias_stddev>0.0000008</bias_stddev>
+          </noise>
+        </z>
+      </angular_velocity>
+      <linear_acceleration>
+        <x>
+          <noise type="gaussian">
+            <mean>0.0</mean>
+            <stddev>1.7e-2</stddev>
+            <bias_mean>0.1</bias_mean>
+            <bias_stddev>0.001</bias_stddev>
+          </noise>
+        </x>
+        <y>
+          <noise type="gaussian">
+            <mean>0.0</mean>
+            <stddev>1.7e-2</stddev>
+            <bias_mean>0.1</bias_mean>
+            <bias_stddev>0.001</bias_stddev>
+          </noise>
+        </y>
+        <z>
+          <noise type="gaussian">
+            <mean>0.0</mean>
+            <stddev>1.7e-2</stddev>
+            <bias_mean>0.1</bias_mean>
+            <bias_stddev>0.001</bias_stddev>
+          </noise>
+        </z>
+      </linear_acceleration>
+    </imu>
+  </sensor>
+</gazebo>
 <gazebo>
   <plugin name="velocity_controller" filename="libgazebo_ros_diff_drive.so">

File: grobot_description/urdf/R1V2/materials.xacro (robot description, xacro)
@@ -1,4 +1,7 @@
 <?xml version="1.0" ?>
 <robot name="R1V2" xmlns:xacro="http://www.ros.org/wiki/xacro" >
+<material name="black">
+  <color rgba="0.000 0.000 0.000 0.700"/>
+</material>
 <material name="silver">
   <color rgba="0.700 0.700 0.700 1.000"/>

Commit message: Fix : Odom TF

File: grobot_description/urdf/R1V2/R1V2.xacro (robot description, xacro)
@@ -2,7 +2,8 @@
 <robot name="R1V2" xmlns:xacro="http://www.ros.org/wiki/xacro">
 <xacro:include filename="$(find grobot_description)/urdf/materials.xacro" />
-<xacro:include filename="$(find grobot_description)/urdf/R1V2.trans" />
+<!-- <xacro:include filename="$(find grobot_description)/urdf/R1V2.trans" /> -->
 <xacro:include filename="$(find grobot_description)/urdf/R1V2.gazebo" />
 <xacro:property name="body_color" value="Gazebo/Grey" />
+<!-- BASE FOOTPRINT -->
 <link name="base_footprint"/>
 <joint name="base_joint" type="fixed">
@@ -11,4 +12,5 @@
   <origin xyz="0 0.0 0.0" rpy="0 0 0.0"/>
 </joint>
+<!-- BASE LINK -->
 <link name="base_link">
   <inertial>
@@ -31,5 +33,6 @@
   </collision>
 </link>
-<link name="right_wheel_1">
+<!-- RIGHT WHEEL -->
+<link name="wheel_right_link">
   <inertial>
     <origin xyz="-6.635167877216963e-06 -0.03788510222333019 2.6177456940168486e-06" rpy="0 0 0"/>
@@ -51,5 +54,12 @@
   </collision>
 </link>
-<link name="left_wheel_1">
+<joint name="wheel_right_joint" type="continuous">
+  <origin xyz="0.19013 -0.260644 0.100803" rpy="0 0 0"/>
+  <parent link="base_link"/>
+  <child link="wheel_right_link"/>
+  <axis xyz="0.0 1.0 0.0"/>
+</joint>
+<!-- LEFT WHEEL -->
+<link name="wheel_left_link">
   <inertial>
     <origin xyz="6.35960602515806e-06 0.03788468935132683 2.6476887081960943e-06" rpy="0 0 0"/>
@@ -71,4 +81,11 @@
   </collision>
 </link>
+<joint name="wheel_left_joint" type="continuous">
+  <origin xyz="0.190619 0.2724 0.100803" rpy="0 0 0"/>
+  <parent link="base_link"/>
+  <child link="wheel_left_link"/>
+  <axis xyz="0.0 1.0 -0.0"/>
+</joint>
+<!-- LIDAR  -->
 <link name="base_scan">
   <inertial>
@@ -90,26 +107,8 @@
   </collision> -->
 </link>
-<joint name="right_wheel_joint" type="continuous">
-  <origin xyz="0.19013 -0.260644 0.100803" rpy="0 0 0"/>
-  <parent link="base_link"/>
-  <child link="right_wheel_1"/>
-  <axis xyz="0.0 1.0 0.0"/>
-</joint>
-<joint name="left_wheel_joint" type="continuous">
-  <origin xyz="0.190619 0.2724 0.100803" rpy="0 0 0"/>
-  <parent link="base_link"/>
-  <child link="left_wheel_1"/>
-  <axis xyz="0.0 1.0 -0.0"/>
-</joint>
 <joint name="lidar_joint" type="fixed">
   <origin xyz="0.0 0.0 0.4" rpy="0 0 3.14159"/>
   <parent link="base_link"/>
   <child link="base_scan"/>
-  <axis xyz="0.0 0.0 1.0"/>
-</joint>
-<joint name="imu_joint" type="fixed">
-  <origin xyz="0.0 0.0 0.2" rpy="0 0 0"/>
-  <parent link="base_link"/>
-  <child link="imu_link"/>
   <axis xyz="0.0 0.0 1.0"/>
 </joint>
@@ -146,4 +145,11 @@
         </sensor>
 </gazebo>
+<!-- IMU -->
+<joint name="imu_joint" type="fixed">
+  <origin xyz="0.0 0.0 0.2" rpy="0 0 0"/>
+  <parent link="base_link"/>
+  <child link="imu_link"/>
+  <axis xyz="0.0 0.0 1.0"/>
+</joint>
 <link name="imu_link"/>
  <gazebo reference="imu_link">
@@ -214,10 +220,11 @@
   </sensor>
 </gazebo>
+<!-- CONTROLLER -->
 <gazebo>
   <plugin name="velocity_controller" filename="libgazebo_ros_diff_drive.so">
     <update_rate>30</update_rate>
     <!-- Wheel Information -->
-    <left_joint>left_wheel_joint</left_joint>
-    <right_joint>right_wheel_joint</right_joint>
+    <left_joint>wheel_left_joint</left_joint>
+    <right_joint>wheel_right_joint</right_joint>
     <wheel_separation>0.650</wheel_separation>
     <wheel_diameter>0.22</wheel_diameter>
@@ -232,7 +239,8 @@
     <publish_odom>true</publish_odom>
     <publish_odom_tf>true</publish_odom_tf>
-    <publish_wheel_tf>false</publish_wheel_tf>
+    <publish_wheel_tf>true</publish_wheel_tf>
   </plugin>
 </gazebo>
+<!-- JOINT STATE -->
 <gazebo>
   <plugin name="grobot_joint_state" filename="libgazebo_ros_joint_state_publisher.so">
@@ -241,6 +249,6 @@
     </ros>
     <update_rate>30</update_rate>
-    <joint_name>left_wheel_joint</joint_name>
-    <joint_name>right_wheel_joint</joint_name>
+    <joint_name>wheel_left_joint</joint_name>
+    <joint_name>wheel_right_joint</joint_name>
   </plugin>
 </gazebo>

Commit message: Add : Gazebo Navigation

File: grobot_description/urdf/R1V2/R1V2.xacro (robot description, xacro)
@@ -34,4 +34,10 @@
 </link>
 <!-- RIGHT WHEEL -->
+<joint name="wheel_right_joint" type="continuous">
+  <origin xyz="0.19013 -0.260644 0.100803" rpy="0 0 0"/>
+  <parent link="base_link"/>
+  <child link="wheel_right_link"/>
+  <axis xyz="0.0 1.0 0.0"/>
+</joint>
 <link name="wheel_right_link">
   <inertial>
@@ -54,11 +60,11 @@
   </collision>
 </link>
-<joint name="wheel_right_joint" type="continuous">
-  <origin xyz="0.19013 -0.260644 0.100803" rpy="0 0 0"/>
-  <parent link="base_link"/>
-  <child link="wheel_right_link"/>
-  <axis xyz="0.0 1.0 0.0"/>
-</joint>
 <!-- LEFT WHEEL -->
+<joint name="wheel_left_joint" type="continuous">
+  <origin xyz="0.190619 0.2724 0.100803" rpy="0 0 0"/>
+  <parent link="base_link"/>
+  <child link="wheel_left_link"/>
+  <axis xyz="0.0 1.0 -0.0"/>
+</joint>
 <link name="wheel_left_link">
   <inertial>
@@ -81,11 +87,11 @@
   </collision>
 </link>
-<joint name="wheel_left_joint" type="continuous">
-  <origin xyz="0.190619 0.2724 0.100803" rpy="0 0 0"/>
-  <parent link="base_link"/>
-  <child link="wheel_left_link"/>
-  <axis xyz="0.0 1.0 -0.0"/>
-</joint>
 <!-- LIDAR  -->
+<joint name="lidar_joint" type="fixed">
+  <origin xyz="0.0 0.0 0.4" rpy="0 0 3.14159"/>
+  <parent link="base_link"/>
+  <child link="base_scan"/>
+  <axis xyz="0.0 0.0 1.0"/>
+</joint>
 <link name="base_scan">
   <inertial>
@@ -94,23 +100,17 @@
     <inertia ixx="0.001" iyy="0.000000" izz="0.000000" ixy="0.001" iyz="0.000000" ixz="0.001"/>
   </inertial>
-  <!-- <visual name="lidar_sensor_visual">
+  <collision>
     <origin xyz="0.0 0.0 0.0" rpy="0 0 0"/>
     <geometry>
-      <mesh filename="file://$(find grobot_description)/meshes/lidar_1.stl" scale="0.001 0.001 0.001"/>
-    </geometry>
-  </visual>
-  <collision name="lidar_sensor_collision">
+      <cylinder length="0.0315" radius="0.055"/>
+    </geometry>
+  </collision>
+  <visual>
     <origin xyz="0.0 0.0 0.0" rpy="0 0 0"/>
     <geometry>
-      <mesh filename="file://$(find grobot_description)/meshes/lidar_1.stl" scale="0.001 0.001 0.001"/>
-    </geometry>
-  </collision> -->
-</link>
-<joint name="lidar_joint" type="fixed">
-  <origin xyz="0.0 0.0 0.4" rpy="0 0 3.14159"/>
-  <parent link="base_link"/>
-  <child link="base_scan"/>
-  <axis xyz="0.0 0.0 1.0"/>
-</joint>
+      <cylinder length="0.0315" radius="0.055"/>
+    </geometry>
+  </visual>
+</link>
 <gazebo reference="base_scan">
         <sensor name="laser" type="ray">

Commit message: Add : Second LIDAR TF

File: grobot_description/urdf/R1V2/R1V2.xacro (robot description, xacro)
@@ -87,7 +87,7 @@
   </collision>
 </link>
-<!-- LIDAR  -->
+<!-- LIDAR RIGHT-->
 <joint name="lidar_joint" type="fixed">
-  <origin xyz="0.0 0.0 0.4" rpy="0 0 3.14159"/>
+  <origin xyz="0.27 -0.27 0.4" rpy="0 0 3.14159"/>
   <parent link="base_link"/>
   <child link="base_scan"/>
@@ -95,4 +95,30 @@
 </joint>
 <link name="base_scan">
+  <inertial>
+    <origin xyz="0.0 0.0 0.0" rpy="0 0 0"/>
+    <mass value="0.114"/>
+    <inertia ixx="0.001" iyy="0.000000" izz="0.000000" ixy="0.001" iyz="0.000000" ixz="0.001"/>
+  </inertial>
+  <collision>
+    <origin xyz="0.0 0.0 0.0" rpy="0 0 0"/>
+    <geometry>
+      <cylinder length="0.0315" radius="0.055"/>
+    </geometry>
+  </collision>
+  <visual>
+    <origin xyz="0.0 0.0 0.0" rpy="0 0 0"/>
+    <geometry>
+      <cylinder length="0.0315" radius="0.055"/>
+    </geometry>
+  </visual>
+</link>
+<!-- LIDAR LEFT-->
+<joint name="lidar_joint2" type="fixed">
+  <origin xyz="0.27 0.27 0.45" rpy="0 0 3.14159"/>
+  <parent link="base_link"/>
+  <child link="base_scan2"/>
+  <axis xyz="0.0 0.0 1.0"/>
+</joint>
+<link name="base_scan2">
   <inertial>
     <origin xyz="0.0 0.0 0.0" rpy="0 0 0"/>
@@ -122,6 +148,6 @@
                     <horizontal>
                         <samples>360</samples>
-                        <min_angle>-3.14</min_angle>
-                        <max_angle>3.14</max_angle>
+                        <min_angle>0.0</min_angle>
+                        <max_angle>4.71</max_angle>
                     </horizontal>
                 </scan>
@@ -142,4 +168,36 @@
                 <output_type>sensor_msgs/LaserScan</output_type>
                 <frame_name>base_scan</frame_name>
+            </plugin>
+        </sensor>
+</gazebo>
+<gazebo reference="base_scan2">
+        <sensor name="laser2" type="ray">
+            <pose> 0 0 0 0 0 0 </pose>
+            <visualize>true</visualize>
+            <update_rate>10</update_rate>
+            <ray>
+                <scan>
+                    <horizontal>
+                        <samples>360</samples>
+                        <min_angle>1.57</min_angle>
+                        <max_angle>6.28</max_angle>
+                    </horizontal>
+                </scan>
+                <range>
+                    <min>0.1</min>
+                    <max>16</max>
+                </range>
+                <noise>
+                  <type>gaussian</type>
+                  <mean>0.0</mean>
+                  <stddev>0.01</stddev>
+                </noise>
+            </ray>
+            <plugin name="scan2" filename="libgazebo_ros_ray_sensor.so">
+                <ros>
+                    <argument>~/out:=scan</argument>
+                </ros>
+                <output_type>sensor_msgs/LaserScan</output_type>
+                <frame_name>base_scan2</frame_name>
             </plugin>
         </sensor>

Commit message: Add : Merge LIDAR TF

File: grobot_description/urdf/R1V2/R1V2.xacro (robot description, xacro)
@@ -139,4 +139,29 @@
   </visual>
 </link>
+<joint name="merged_lidar_joint" type="fixed">
+  <origin xyz="0.0 0.0 0.45" rpy="0 0 3.14159"/>
+  <parent link="base_link"/>
+  <child link="merged_base_scan"/>
+  <axis xyz="0.0 0.0 1.0"/>
+</joint>
+<link name="merged_base_scan">
+  <inertial>
+    <origin xyz="0.0 0.0 0.0" rpy="0 0 0"/>
+    <mass value="0.114"/>
+    <inertia ixx="0.001" iyy="0.000000" izz="0.000000" ixy="0.001" iyz="0.000000" ixz="0.001"/>
+  </inertial>
+  <!-- <collision>
+    <origin xyz="0.0 0.0 0.0" rpy="0 0 0"/>
+    <geometry>
+      <cylinder length="0.0315" radius="0.055"/>
+    </geometry>
+  </collision> -->
+  <visual>
+    <origin xyz="0.0 0.0 0.0" rpy="0 0 0"/>
+    <geometry>
+      <cylinder length="0.0315" radius="0.055"/>
+    </geometry>
+  </visual>
+</link>
 <gazebo reference="base_scan">
         <sensor name="laser" type="ray">
@@ -148,5 +173,5 @@
                     <horizontal>
                         <samples>360</samples>
-                        <min_angle>-3.14</min_angle>
+                        <min_angle>0</min_angle>
                         <max_angle>3.14</max_angle>
                     </horizontal>
@@ -182,5 +207,5 @@
                         <samples>360</samples>
                         <min_angle>-3.14</min_angle>
-                        <max_angle>3.14</max_angle>
+                        <max_angle>0</max_angle>
                     </horizontal>
                 </scan>

Commit message: Change Lidar joint URDF

File: grobot_description/urdf/R1V2/R1V2.xacro (robot description, xacro)
@@ -89,5 +89,5 @@
 <!-- LIDAR RIGHT-->
 <joint name="lidar_joint" type="fixed">
-  <origin xyz="0.27 -0.27 0.4" rpy="0 0 3.14159"/>
+  <origin xyz="0.37 -0.265 0.26" rpy="0 0 3.14159"/>
   <parent link="base_link"/>
   <child link="base_scan"/>
@@ -115,5 +115,5 @@
 <!-- LIDAR LEFT-->
 <joint name="lidar_joint2" type="fixed">
-  <origin xyz="0.27 0.27 0.45" rpy="0 0 3.14159"/>
+  <origin xyz="0.37 0.265 0.34" rpy="0 0 3.14159"/>
   <parent link="base_link"/>
   <child link="base_scan2"/>

Commit message: Fix : LIDAR Frame Orientation

File: grobot_description/urdf/R1V2/R1V2.xacro (robot description, xacro)
@@ -89,5 +89,5 @@
 <!-- LIDAR RIGHT-->
 <joint name="lidar_joint" type="fixed">
-  <origin xyz="0.37 -0.265 0.26" rpy="0 0 3.14159"/>
+  <origin xyz="0.37 -0.265 0.26" rpy="0 0 2.35619"/>
   <parent link="base_link"/>
   <child link="base_scan"/>
@@ -115,5 +115,5 @@
 <!-- LIDAR LEFT-->
 <joint name="lidar_joint2" type="fixed">
-  <origin xyz="0.37 0.265 0.34" rpy="0 0 3.14159"/>
+  <origin xyz="0.37 0.265 0.34" rpy="0 0 3.92699"/>
   <parent link="base_link"/>
   <child link="base_scan2"/>

Commit message: Temp commit NUC

File: grobot_description/urdf/R1V2/R1V2.xacro (robot description, xacro)
@@ -232,5 +232,5 @@
 <!-- IMU -->
 <joint name="imu_joint" type="fixed">
-  <origin xyz="0.0 0.0 0.2" rpy="0 0 0"/>
+  <origin xyz="0.35 0.0 0.2" rpy="0 0 0"/>
   <parent link="base_link"/>
   <child link="imu_link"/>

Commit message: FEAT : xacro updated and feat process node

File: grobot_description/urdf/R1V2/R1V2.xacro (robot description, xacro)
@@ -229,4 +229,11 @@
         </sensor>
 </gazebo>
+<!-- CAMERA LINK -->
+<link name="camera_link"/>
+<joint name="camera_joint" type="fixed">
+  <parent link="base_link"/>
+  <child link="camera_link"/>
+  <origin xyz="0.11565 0.005 0.2230" rpy="0 0 0"/>
+</joint>
 <!-- IMU -->
   <!-- <origin xyz="0.35 0.0 0.2" rpy="0 0 0"/> -->

File: grobot_description/urdf/grobot/grobot.xacro (robot description, xacro)
@@ -14,5 +14,5 @@
 <link name="camera_link"/>
 <joint name="camera_joint" type="fixed">
-  <parent link="imu_link"/>
+  <parent link="base_link"/>
   <child link="camera_link"/>
   <origin xyz="0 0.0 0.0" rpy="0 0 0.0"/>
